File: projecte_mise.kicad_sch (KiCad schematic)
At the start: 16 parts, among them IC1 MSP430FR2355TPT, J1 conn_DFrobot, SW1 SW_Push, U1 LMV324, Y2 Crystal

Commit message: Add files via upload
Parts:
- removed C3: 12pF, symbol Device:C_Small
- added C1: 12pF, Capacitor_SMD:C_0805_2012Metric_Pad1.18x1.45mm_HandSolder, symbol Device:C_Small
- added CCOUPLING2, CCOUPLING4: 100nF, Capacitor_SMD:C_0805_2012Metric_Pad1.18x1.45mm_HandSolder, symbol Device:C_Small
- added CSBW: 2.2nF, Capacitor_SMD:C_0805_2012Metric_Pad1.18x1.45mm_HandSolder, symbol Device:C_Small
- added J2: ESP01, symbol Connector_Generic:Conn_02x04_Odd_Even
- added J3: SBW, symbol Connector:Screw_Terminal_01x03
- added R8: R, symbol Device:R
- added RV1, RV2: Device_R_POT, MiSE:Trimmer_MiSE, symbol MiSE:R_POT-Device
- C4: footprint (none) -> Capacitor_SMD:C_0805_2012Metric_Pad1.18x1.45mm_HandSolder
Connections:
- net RESET is gone; now on net RESET/TDIO: R2.2, SW1.1
- net VCC is gone; now on net +3.3V: J1.1 (Pin_1), J1.2 (Pin_2), LCD1.1 (VDD), R2.1, R4.1
- net GND: now also IC1.1 (P1.2/UCB0SIMO/UCB0SDA/TB0TRG/OA0-/A2/VEREF-), IC1.7 (DVSS), C1.2, CCOUPLING2.2, CCOUPLING4.2, CSBW.2, J2.7 (Pin_7), J3.1 (Pin_1), RV1.3, RV2.3
- net RXD: now also J2.1 (Pin_1)
- net TXD: now also J2.8 (Pin_8)
- net XIN: now also C1.1
- net +3.3V: now reaches R7.1
- net +3.3V: now also IC1.3 (P1.0/UCB0STE/SMCLK/COMP0.0/A0/VEREF+), IC1.6 (DVCC), R5.1, CCOUPLING2.1, CCOUPLING4.1, J2.2 (Pin_2)
- net A9: now reaches R7.2
- net A9: now also IC1.42 (P5.1/TB2.2/MFM.TX/A9), RV1.2
- net P5.2: now reaches LCD1.5 (RST)
- net P5.2: now also IC1.41 (P5.2/TB2CLK/A10)
- net A8: now reaches R5.2
- net A8: now also IC1.43 (P5.0/TB2.1/MFM.RX/A8), RV2.2
- net SBWTCK: now reaches IC1.4 (TEST/SBWTCK)
- net SBWTCK: now also J3.2 (Pin_2)
- net RESET/TDIO: now reaches IC1.5 (~{RST}/NMI/SBWTDIO)
- net RESET/TDIO: now also CSBW.1, J3.3 (Pin_3)
- new net C_ENABLE: J2.6 (Pin_6)
- no-connect marks 0 -> 6
Other:
- note added: "COUPLING POWER"
- note added: "COUPLING VREF"
- note added: "Es fa servir la comunicacio I2C PIN 9 I 11 PINS:3,5,7 (SCLK.MISO,MOSI) Son comunicacio SPI MODUL ULTRASONS (TRIGGER/ECHO) ??"
- note added: "PIN ENABLE : GPIO"
- note added: "PINES DESTINADOS A GPIO: P1.0: RESET DISPLAY LCD"
- note added: "SBW"
- note added: "TRIMMER CONFIGURACIO ANALOGICA O DIGITAL?"
- moved on the sheet: IC1, J1, R2, R3, R4, R5, R6, R7, S1, U1A, U1B
