File: Rossend_Cera_Bethany_Quintero_MISE_V3.kicad_pcb (KiCad board)
At the start: 2 copper layers, 80 x 75 mm, 31 parts, among them IC1 MSP430FR2355TPT, J1 Conn_01x02_Pin, J2 conn_DFrobot, J3 SBW, J4 ESP01, J5 Conn_01x02_Pin, J6 Conn_01x03_Pin, J7 Conn_01x03_Pin, SW1 SW_Push, U1 LMV324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

Commit message: Add files via upload
Parts:
- moved J1 21.9 mm to (117.2, 103.8), turned to 90 degrees
- moved U1 16.9 mm to (125.0, 82.0), turned to -90 degrees
- moved R_SDA1 10.1 mm to (104.2, 101.5), turned to 180 degrees
- moved R_SCL1 9.60 mm to (104.2, 107.5), turned to 180 degrees
- moved J5 6.02 mm to (127.2, 103.2), turned to -90 degrees
- moved J6 4.72 mm to (105.2, 112.0)
- moved J4 0.56 mm to (125.0, 100.5)
Connections:
- IC1 pad 12: /SD- -> SCL
- IC1 pad 13: /SD+ -> SDA
- IC1 pad 44: /GPIO_R -> /GPIO_T
- IC1 pad 45: /GPIO_B -> /GPIO_R
- IC1 pad 46: /GPIO_T -> /GPIO_B
- R_SCL1 pad 2: /SD- -> SCL
- R_SDA1 pad 2: /SD+ -> SDA
Routing:
- net SCL: track 0.00 -> 91.2 mm, vias 0 -> 1
- net SDA: track 0.00 -> 75.7 mm
- net G(P2.4): track 0.00 -> 23.1 mm
- net Analog_outTB: track 0.00 -> 15.9 mm, vias 0 -> 1
- net RXD: track 0.00 -> 10.8 mm, vias 0 -> 1
- net TXD: track 0.00 -> 10.6 mm
- net /GPIO_T: track 0.00 -> 9.81 mm
- net C_ENABLE: track 0.00 -> 6.10 mm
- net Net-(U1D--): track 0.00 -> 6.04 mm
- net /GPIO_R: track 0.00 -> 3.77 mm
- net /GPIO_B: track 0.00 -> 3.77 mm
- net Net-(U1C-+): track 0.00 -> 3.25 mm
- net GND: vias 38 -> 26

Commit message: Add files via upload
Parts:
- U1: footprint MiSE:LMV324 -> MiSE:SOIC127P600X175-14N
- moved RV2 63.2 mm to (105.4, 63.3), turned to 0 degrees
- moved R3 63.1 mm to (109.5, 58.4), turned to -90 degrees
- moved R2 62.5 mm to (115.6, 58.4), turned to 90 degrees
- moved J7 60.4 mm to (91.7, 106.2), turned to 180 degrees
- moved S1 56.5 mm to (92.2, 115.5), turned to 90 degrees
- moved RV1 55.1 mm to (113.8, 63.3)
- moved J6 54.0 mm to (101.6, 58.2), turned to -90 degrees
- moved SW1 48.1 mm to (129.6, 113.0), turned to 90 degrees
- moved R1 46.7 mm to (130.1, 117.3), turned to 180 degrees
- moved CSBW1 42.8 mm to (130.8, 101.6), turned to 90 degrees
- moved R9 42.0 mm to (116.3, 113.0)
- moved R8 41.0 mm to (119.9, 108.7), turned to -90 degrees
- moved R4 40.3 mm to (116.2, 108.9)
- moved R7 39.5 mm to (123.1, 108.7), turned to 90 degrees
- moved R6 39.3 mm to (123.2, 113.0)
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Routing:
- net Analog_out_RL: track 0.00 -> 51.3 mm, vias 0 -> 2
- net A8: track 0.00 -> 49.9 mm, vias 0 -> 1
- net A9: track 0.00 -> 41.3 mm, vias 0 -> 1
- net RESET/TDIO: track 0.00 -> 40.8 mm
- net SCL: track 91.2 -> 50.6 mm, vias 1 -> 0
- net SDA: track 75.7 -> 39.8 mm
- net /SBWTCK: track 0.00 -> 19.7 mm
- net Analog_outTB: track 15.9 -> 35.0 mm, vias 1 -> 0
- net Net-(U1A-+): track 0.00 -> 16.9 mm
- net ECHO: track 0.00 -> 15.7 mm
- net Net-(U1B--): track 0.00 -> 12.2 mm
- net /GPIO_B: track 3.77 -> 15.5 mm
- net Net-(U1D--): track 6.04 -> 16.8 mm, vias 0 -> 2
- net TRIGGER: track 0.00 -> 10.4 mm
- net Net-(U1C-+): track 3.25 -> 12.5 mm
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
Commit message: Add files via upload
Parts:
- moved J5 53.4 mm to (115.7, 72.0), turned to 90 degrees
- moved J4 49.7 mm to (117.8, 75.8), turned to -90 degrees
- moved R_SCL1 26.9 mm to (97.2, 91.8), turned to -90 degrees
- moved R_SDA1 25.4 mm to (97.2, 96.8), turned to 90 degrees
- moved J6 17.5 mm to (97.0, 75.1), turned to 180 degrees
- moved J1 16.0 mm to (143.9, 77.5), turned to 180 degrees
- moved SW1 14.1 mm to (128.4, 99.0), turned to 0 degrees
- moved CSBW1 9.59 mm to (128.9, 92.2), turned to -90 degrees
- moved J3 8.75 mm to (135.1, 91.9)
- moved R7 8.30 mm to (115.8, 112.6)
- moved R5 6.18 mm to (122.8, 107.6), turned to -90 degrees
- moved R9 5.28 mm to (119.0, 117.6)
- moved R6 4.48 mm to (123.7, 117.5)
- moved R1 4.40 mm to (132.0, 113.4)
- moved J7 4.39 mm to (92.2, 101.8), turned to 0 degrees
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Connections:
- IC1 pad 11: G(P2.4) -> unconnected-(IC1-P2.4/COMP1.1-Pad11)
- IC1 pad 36: unconnected-(IC1-P3.6/OA3--Pad36) -> G(P2.4)
- IC1 pad 37: unconnected-(IC1-P3.5/OA3O-Pad37) -> DF_Robot
- IC1 pad 38: /GPIO_L -> /GPIO_R
- IC1 pad 44: /GPIO_T -> /GPIO_L
- IC1 pad 45: /GPIO_R -> /GPIO_T
- IC1 pad 47: DF_Robot -> unconnected-(IC1-P3.0/MCLK-Pad47)
Routing:
- net SDA: track 39.8 -> 109.1 mm, vias 0 -> 2
- net SCL: track 50.6 -> 111.3 mm, vias 0 -> 2
- net Rst_n_display: track 0.00 -> 40.8 mm, vias 0 -> 1
- net DF_Robot: track 6.50 -> 32.0 mm
- net C_ENABLE: track 0.00 -> 20.0 mm, vias 0 -> 1
- net A9: track 41.3 -> 59.3 mm
- net A8: track 49.9 -> 64.2 mm
- net Net-(U1B--): track 12.2 -> 25.7 mm, vias 0 -> 2
- net G(P2.4): track 22.6 -> 12.1 mm
- net /GPIO_B: track 15.5 -> 5.10 mm
- net Analog_outTB: track 35.0 -> 45.2 mm, vias 0 -> 2
- net TXD: track 5.19 -> 15.1 mm
- net Net-(U1C-+): track 12.5 -> 21.9 mm
- net GND: track 0.00 -> 8.56 mm, vias 30 -> 4
- net XIN: track 6.86 -> 0.00 mm
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- added copper zone on F.Cu, net +3.3V
- added copper zone on B.Cu, net GND
- removed copper zone on F.Cu, net GND

Commit message: Add files via upload
Parts:
- J1, J5: footprint Connector_PinHeader_1.00mm:PinHeader_1x02_P1.00mm_Vertical -> Connector_PinHeader_2.54mm:PinHeader_1x02_P2.54mm_Vertical
- J3, J6, J7: footprint Connector_PinHeader_1.00mm:PinHeader_1x03_P1.00mm_Vertical -> Connector_PinHeader_2.54mm:PinHeader_1x03_P2.54mm_Vertical
- J4: footprint Connector_PinHeader_1.00mm:PinHeader_2x04_P1.00mm_Vertical -> Connector_PinHeader_2.54mm:PinHeader_2x04_P2.54mm_Vertical
- moved J5 10.8 mm to (125.4, 67.4)
- moved R4 10.7 mm to (115.8, 117.6), turned to -90 degrees
- moved J1 9.53 mm to (134.4, 76.8)
- moved J3 8.77 mm to (129.8, 98.9), turned to 90 degrees
- moved J6 7.22 mm to (97.0, 67.9)
- moved CCOUPLING2 4.87 mm to (130.2, 90.2), turned to 90 degrees
- moved J4 4.56 mm to (121.1, 72.7)
- moved SW1 4.12 mm to (128.8, 103.0)
- moved CSBW1 3.00 mm to (130.3, 94.8), turned to 0 degrees
- moved C1 2.27 mm to (134.0, 87.5)
- moved C2 1.99 mm to (133.9, 81.0)
- moved J7 1.56 mm to (91.6, 100.4)
- moved R1 1.28 mm to (131.0, 114.2), turned to 90 degrees
- moved R5 0.80 mm to (123.6, 107.7)
- moved Y1 0.43 mm to (127.0, 85.2)
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Connections:
- IC1 pad 44: /GPIO_L -> /GPIO_T
- IC1 pad 45: /GPIO_T -> /GPIO_L
Routing:
- net +3.3V: track 0.00 -> 27.5 mm, vias 0 -> 1
- net GND: track 8.56 -> 33.8 mm, vias 4 -> 10
- net Net-(U1A-+): track 12.1 -> 34.4 mm
- net TXD: track 15.1 -> 29.0 mm
- net SDA: track 109.1 -> 96.4 mm
- net XIN: track 0.00 -> 11.5 mm
- net RXD: track 15.4 -> 26.6 mm
- net A9: track 59.3 -> 66.8 mm
- net Net-(U1B--): track 25.7 -> 18.2 mm
- net XOUT: track 5.31 -> 12.0 mm
- net C_ENABLE: track 20.0 -> 25.9 mm
- net Analog_outTB: track 45.2 -> 51.0 mm, vias 2 -> 1
- net RESET/TDIO: track 35.0 -> 40.7 mm
- net A8: track 64.2 -> 69.9 mm
- net /GPIO_T: track 14.8 -> 20.4 mm, vias 0 -> 2
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