File: Rossend_Cera_Bethany_Quintero_MISE_V3.kicad_sch (KiCad schematic)
At the start: 38 parts, among them IC1 MSP430FR2355TPT, J2 conn_DFrobot, J3 SBW, J4 ESP01, SW1 SW_Push, U1 LMV324, U2 LMV324, Y1 Crystal

Commit message: Add files via upload
Parts:
- removed TP1, TP10, TP11, TP3, TP4, TP5, TP6, TP7, TP8, TP9: TestPoint, Connector_PinHeader_1.00mm:PinHeader_1x01_P1.00mm_Vertical, symbol Connector:TestPoint
- removed U2: LMV324, symbol Amplifier_Operational:LMV324
- added J1, J5: Conn_01x02_Pin, Connector_PinHeader_1.00mm:PinHeader_1x02_P1.00mm_Vertical, symbol Connector:Conn_01x02_Pin
- added J6, J7: Conn_01x03_Pin, Connector_PinHeader_1.00mm:PinHeader_1x03_P1.00mm_Vertical, symbol Connector:Conn_01x03_Pin
- added unit 5 of U1
- added unit 3 of U1
- added unit 4 of U1
- U1: footprint (none) -> MiSE:LMV324
Connections:
- net +3.3V: now also U1.4 (V+)
- net A8: now also IC1.33 (P1.5/UCA0CLK/TMS/OA1O/A5), J6.1 (Pin_1); no longer IC1.43 (P5.0/TB2.1/MFM.RX/A8)
- net A9: now also IC1.34 (P1.4/UCA0STE/TCK/A4), J6.2 (Pin_2); no longer IC1.42 (P5.1/TB2.2/MFM.TX/A9)
- net Analog_outTB: now also U1.2 (-), U1.5 (+), J7.1 (Pin_1); no longer U1.3 (+), U1.6 (-)
- net Analog_out_RL: now also J7.2 (Pin_2), U1.12 (+), U1.9 (-)
- net C_ENABLE: now also IC1.15 (P4.4/UCB1STE); no longer IC1.37 (P3.5/OA3O)
- net GND: now also J6.3 (Pin_3), J7.3 (Pin_3), U1.11 (V-)
- net GPIO_B: now also U1.7; no longer U1.1
- net GPIO_L: now also U1.14
- net GPIO_R: now also U1.8
- net GPIO_T: now also U1.1; no longer U1.7
- net RXD: now also IC1.23 (P4.3/UCA1TXD/UCA1SIMO/~{UCA1TXD}), J5.2 (Pin_2); no longer IC1.31 (P1.7/UCA0TXD/UCA0SIMO/TB0.2/TDO/OA1+/A7/VREF+)
- net Rst_n_display: now also IC1.14 (P4.5/UCB1CLK); no longer IC1.10 (P2.5/COMP1.0)
- net SCL: now also J1.1 (Pin_1)
- net SDA: now also J1.2 (Pin_2)
- net TXD: now also IC1.24 (P4.2/UCA1RXD/UCA1SOMI/~{UCA1RXD}), J5.1 (Pin_1); no longer IC1.32 (P1.6/UCA0RXD/UCA0SOMI/TB0.1/TDI/TCLK/OA1-/A6)
- net at R7.2, R8.1: now also U1.10 (+)
- net at R8.2, R9.1: now also U1.13 (-)
- net at R5.2, R6.1: now also U1.6 (-); no longer U1.2 (-)
- net at R4.2, R5.1: now also U1.3 (+); no longer U1.5 (+)
- no-connect marks 33 -> 35

Commit message: Add files via upload
Connections:
- net GPIO_B: now also IC1.46 (P3.1/OA2O); no longer IC1.45 (P3.2/OA2-)
- net GPIO_R: now also IC1.45 (P3.2/OA2-); no longer IC1.44 (P3.3/OA2+)
- net GPIO_T: now also IC1.44 (P3.3/OA2+); no longer IC1.46 (P3.1/OA2O)
Changed lines of the file:
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@@
     (effects (font (size 2 2) (thickness 0.4) bold) (justify left bottom))
   )
-  (label "GPIO_T" (at 144.78 22.86 90) (fields_autoplaced)
+  (label "GPIO_R" (at 147.32 22.86 90) (fields_autoplaced)
     (effects (font (size 1.27 1.27)) (justify left bottom))
   )
@@
     (effects (font (size 1.27 1.27)) (justify left bottom))
   )
-  (label "GPIO_R" (at 149.86 22.86 90) (fields_autoplaced)
+  (label "GPIO_T" (at 149.86 22.86 90) (fields_autoplaced)
     (effects (font (size 1.27 1.27)) (justify left bottom))
   )
@@
     (effects (font (size 1.27 1.27)) (justify left bottom))
   )
-  (label "GPIO_B" (at 147.32 22.86 90) (fields_autoplaced)
+  (label "GPIO_B" (at 144.78 22.86 90) (fields_autoplaced)
     (effects (font (size 1.27 1.27)) (justify left bottom))
   )

Commit message: Add files via upload
Parts:
- U1: footprint MiSE:LMV324 -> MiSE:SOIC127P600X175-14N
Other:
- note added: "Configuració TRIMMER"
- note added: "Connector WIFI"
- note added: "Joystick Right & Left"
- note added: "Joystick Top & Bottom"
- note added: "Oscillador"
- note added: "PINES DESTINADOS A GPIO: P2.1.TRIGGER P2.2.LED 1. P2.3 LED 2. P2.4.GPIO GENERICO P2.5.RESET DISPLAY LCD P3.0: Habilitació joystick P3.1: Arriba P3.2: Abajo P3.3:Derecha P3.4:Izquierda P3.5: Chip enable Modulo wifi TIMER: TB1.1:ECHO Connector Robot: Es fa servir la comunicacio I2C PIN 9 I 11 PINS:3,5,7 (SCLK.MISO,MOSI) Son comunicacio SPI MODUL ULTRASONS (TRIGGER/ECHO) ??"
- note removed: "Es fa servir la comunicacio I2C PIN 9 I 11 PINS:3,5,7 (SCLK.MISO,MOSI) Son comunicacio SPI MODUL ULTRASONS (TRIGGER/ECHO) ??"
- note removed: "PINES DESTINADOS A GPIO: P2.1.TRIGGER P2.2.LED 1. P2.3 LED 2. P2.4.GPIO GENERICO P2.5.RESET DISPLAY LCD P3.0: Habilitació joystick P3.1: Arriba P3.2: Abajo P3.3:Derecha P3.4:Izquierda P3.5: Chip enable Modulo wifi TIMER: TB1.1:ECHO"
- note removed: "TRIMMER CONFIGURACIO ANALOGICA O DIGITAL?"
- note removed: "oscillador"
- company: (none) -> Universitat de Barcelona
- title: (none) -> Robot Controller
- moved on the sheet: C1, C2, CCOUPLING1, CCOUPLING2, CSBW1, IC1, J1, J2, J3, J4, J5, J6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

Commit message: Add files via upload
Connections:
- net DF_Robot: now also IC1.37 (P3.5/OA3O); no longer IC1.47 (P3.0/MCLK)
- net G(P2.4): now also IC1.36 (P3.6/OA3-); no longer IC1.11 (P2.4/COMP1.1)
- net GPIO_L: now also IC1.44 (P3.3/OA2+); no longer IC1.38 (P3.4/SMCLK)
- net GPIO_R: now also IC1.38 (P3.4/SMCLK); no longer IC1.45 (P3.2/OA2-)
- net GPIO_T: now also IC1.45 (P3.2/OA2-); no longer IC1.44 (P3.3/OA2+)
Other:
- moved on the sheet: R_SCL1

Commit message: Add files via upload
Parts:
- J1, J5: footprint Connector_PinHeader_1.00mm:PinHeader_1x02_P1.00mm_Vertical -> Connector_PinHeader_2.54mm:PinHeader_1x02_P2.54mm_Vertical
- J3, J6, J7: footprint Connector_PinHeader_1.00mm:PinHeader_1x03_P1.00mm_Vertical -> Connector_PinHeader_2.54mm:PinHeader_1x03_P2.54mm_Vertical
- J4: footprint Connector_PinHeader_1.00mm:PinHeader_2x04_P1.00mm_Vertical -> Connector_PinHeader_2.54mm:PinHeader_2x04_P2.54mm_Vertical
Connections:
- net GPIO_L: now also IC1.45 (P3.2/OA2-); no longer IC1.44 (P3.3/OA2+)
- net GPIO_T: now also IC1.44 (P3.3/OA2+); no longer IC1.45 (P3.2/OA2-)
Changed lines of the file:
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@@
     (effects (font (size 1.27 1.27)) (justify left bottom))
   )
-  (label "GPIO_T" (at 144.272 18.923 90) (fields_autoplaced)
+  (label "GPIO_T" (at 146.812 18.288 90) (fields_autoplaced)
     (effects (font (size 1.27 1.27)) (justify left bottom))
   )
@@
     (effects (font (size 1.27 1.27)) (justify left bottom))
   )
-  (label "GPIO_L" (at 146.812 18.288 90) (fields_autoplaced)
+  (label "GPIO_L" (at 144.272 18.923 90) (fields_autoplaced)
     (effects (font (size 1.27 1.27)) (justify left bottom))
   )
@@
       (effects (font (size 1.27 1.27)))
     )
-    (property "Footprint" "Connector_PinHeader_1.00mm:PinHeader_1x02_P1.00mm_Vertical" (at 14.351 33.274 0)
+    (property "Footprint" "Connector_PinHeader_2.54mm:PinHeader_1x02_P2.54mm_Vertical" (at 14.351 33.274 0)
       (effects (font (size 1.27 1.27)) hide)
     )
@@
       (effects (font (size 1.27 1.27)))
     )
-    (property "Footprint" "Connector_PinHeader_1.00mm:PinHeader_1x03_P1.00mm_Vertical" (at 14.478 47.244 0)
+    (property "Footprint" "Connector_PinHeader_2.54mm:PinHeader_1x03_P2.54mm_Vertical" (at 14.478 47.244 0)
       (effects (font (size 1.27 1.27)) hide)
     )
@@
       (effects (font (size 1.27 1.27)))
     )
-    (property "Footprint" "Connector_PinHeader_1.00mm:PinHeader_2x04_P1.00mm_Vertical" (at 151.892 180.086 0)
+    (property "Footprint" "Connector_PinHeader_2.54mm:PinHeader_2x04_P2.54mm_Vertical" (at 151.892 180.086 0)
       (effects (font (size 1.27 1.27)) hide)
     )
@@
       (effects (font (size 1.27 1.27)))
     )
-    (property "Footprint" "Connector_PinHeader_1.00mm:PinHeader_1x03_P1.00mm_Vertical" (at 33.528 40.64 0)
+    (property "Footprint" "Connector_PinHeader_2.54mm:PinHeader_1x03_P2.54mm_Vertical" (at 33.528 40.64 0)
       (effects (font (size 1.27 1.27)) hide)
     )
@@
       (effects (font (size 1.27 1.27)))
     )
-    (property "Footprint" "Connector_PinHeader_1.00mm:PinHeader_1x02_P1.00mm_Vertical" (at 14.097 21.59 0)
+    (property "Footprint" "Connector_PinHeader_2.54mm:PinHeader_1x02_P2.54mm_Vertical" (at 14.097 21.59 0)
       (effects (font (size 1.27 1.27)) hide)
     )
@@
       (effects (font (size 1.27 1.27)))
     )
-    (property "Footprint" "Connector_PinHeader_1.00mm:PinHeader_1x03_P1.00mm_Vertical" (at 51.308 108.966 0)
-      (effects (font (size 1.27 1.27)) hide)
-    )
+    (property "Footprint" "Connector_PinHeader_2.54mm:PinHeader_1x03_P2.54mm_Vertical" (at 51.308 108.966 0)
+      (effects (font (size 1.27 1.27)) hide)
+    )
